File: GreenNet/GreenNet.kicad_pcb (KiCad board)
At the start: 4 copper layers, 95 parts, among them IC5 BQ24250RGER, IC6 NCP186AMX330TAG, Q3 IRF9358TRPBF, Q4 SI3932DV-T1-GE3, Q5 SI3993CDV-T1-GE3, U1 ESP32-S3-WROOM-1-N16R2, U2 USB_C_Receptacle_12P, U3 USB_C_Receptacle_12P, U4 CP2102N-A02-GQFN28, U5 BME280, U6 CYPD3177-24LQXQT, U7 LTR-303ALS-01

Commit message: significant progress
Parts:
- removed D11, D6, D8, D9: Green, LED_SMD:LED_0805_2012Metric
- removed D5: Yellow, LED_SMD:LED_0805_2012Metric
- removed TP1, TP10, TP11, TP12, TP13, TP14, TP15, TP16, TP17, TP18, TP19, TP2, TP20, TP21, TP22, TP23, TP24, TP4, TP6, TP7, TP8, TP9: TestPoint, AA_TestPoints:RCWCTE
- added BT1: Battery_Cell, AA_Connectors:BH18650PC, F.Cu at (150.6, 153.0)
- added C21: 2.2u, Capacitor_SMD:C_0805_2012Metric, F.Cu at (99.5, 136.0)
- added C22: 1u, Capacitor_SMD:C_0805_2012Metric, F.Cu at (99.5, 133.0)
- added C29: 33n, Capacitor_SMD:C_0805_2012Metric, F.Cu at (99.5, 130.0)
- added C30: 22u, Capacitor_SMD:C_0805_2012Metric, F.Cu at (99.5, 127.0)
- added C31: 1u, Capacitor_SMD:C_0805_2012Metric, F.Cu at (99.5, 124.0)
- added C32: 1u, Capacitor_SMD:C_0805_2012Metric, F.Cu at (99.5, 121.0)
- added Connected: Green, LED_SMD:LED_0805_2012Metric, F.Cu at (70.8, 76.7)
- added Connected: Green, LED_SMD:LED_0805_2012Metric, F.Cu at (70.8, 103.8)
- added D13: Yellow, LED_SMD:LED_0805_2012Metric, F.Cu at (117.9, 120.8)
- added D14: D5V0M1U2S9, AA_Diodes:D5V0M1U2S9Q, F.Cu at (125.8, 71.1)
- added D15: D5V0M1U2S9, AA_Diodes:D5V0M1U2S9Q, F.Cu at (125.8, 69.1)
- added H1: MountingHole_Pad, MountingHole:MountingHole_2.5mm_Pad, F.Cu at (72.0, 36.5)
- added H2: MountingHole_Pad, MountingHole:MountingHole_2.5mm_Pad, F.Cu at (58.0, 44.0)
- added H3: MountingHole_Pad, MountingHole:MountingHole_2.5mm_Pad, F.Cu at (58.0, 50.6)
- added H4: MountingHole_Pad, MountingHole:MountingHole_2.5mm_Pad, F.Cu at (58.0, 57.1)
- added J1: Conn_01x03_Pin, AA_Connectors:61300311121, F.Cu at (121.5, 89.5)
- added J2: 3_Pin_Conn, AA_Connectors:61300311121, F.Cu at (158.8, 85.2)
- added J3: 3_Pin_Conn, AA_Connectors:61300311121, F.Cu at (158.8, 81.0)
- added J4: Conn_01x04_Pin, AA_Connectors:61300411121, F.Cu at (142.5, 86.2)
- added J5: 3_Pin_Conn, AA_Connectors:61300311121, F.Cu at (158.8, 76.8)
- added J6: Conn_01x14_Pin, AA_Connectors:CONN_PH1-14-UA_ADM, F.Cu at (166.0, 75.9)
- added L1: 1u, Inductor_SMD:L_0805_2012Metric, F.Cu at (106.8, 133.5)
- added Q6: 2N7002K, Package_TO_SOT_SMD:SOT-23, F.Cu at (123.7, 85.0)
- added Q7: 2N7002K, Package_TO_SOT_SMD:SOT-23, F.Cu at (142.1, 91.7)
- added Q8: MMDT3904, Package_TO_SOT_SMD:SOT-363_SC-70-6, F.Cu at (138.8, 46.5)
- added R17: 5.6k, Resistor_SMD:R_0805_2012Metric, F.Cu at (112.3, 122.6)
- added R21: 12k, Resistor_SMD:R_0805_2012Metric, F.Cu at (112.3, 119.7)
- added R26: 1.3k, Resistor_SMD:R_0805_2012Metric, F.Cu at (112.4, 127.8)
- added R27: 150R, Resistor_SMD:R_0805_2012Metric, F.Cu at (117.4, 124.5)
- added R28: 10k, Resistor_SMD:R_0805_2012Metric, F.Cu at (179.4, 52.8)
- added R29: 10k, Resistor_SMD:R_0805_2012Metric, F.Cu at (179.4, 49.8)
- added R30: 10k, Resistor_SMD:R_0805_2012Metric, F.Cu at (175.0, 61.6)
- added R31: 10k, Resistor_SMD:R_0805_2012Metric, F.Cu at (175.0, 58.6)
- added R32: 10k, Resistor_SMD:R_0805_2012Metric, F.Cu at (175.0, 55.7)
- added R33: 10k, Resistor_SMD:R_0805_2012Metric, F.Cu at (175.0, 52.8)
- added R34: 10k, Resistor_SMD:R_0805_2012Metric, F.Cu at (175.0, 49.8)
- added Recieve: Green, LED_SMD:LED_0805_2012Metric, F.Cu at (75.8, 103.8)
- added SW1: SW_MEC_5E, AA_Switches:18259106, F.Cu at (136.2, 76.2)
- added SW3: SW_MEC_5E, AA_Switches:18259106, F.Cu at (136.2, 67.1)
- added Suspended: Yellow, LED_SMD:LED_0805_2012Metric, F.Cu at (73.2, 103.8)
- added TH1: R_{0}= 10K, B = 3470K, AA_Resistors:MF52A2103J3470, F.Cu at (108.0, 114.8)
- added Transmit: Green, LED_SMD:LED_0805_2012Metric, F.Cu at (78.2, 103.8)
- C10, C6, C7, C8, C9, D4, IC5, R15, R18, R19, R7, R8, U4, U6: moved to B.Cu
- moved U5 122.3 mm to (103.3, 40.5), turned to 180 degrees
- moved U7 121.2 mm to (113.4, 27.8), turned to 180 degrees
- moved C28 120.3 mm to (112.7, 34.7), turned to 180 degrees
- moved C27 116.9 mm to (112.7, 37.7), turned to 180 degrees
- moved IC5 113.5 mm to (98.8, 98.8), turned to 180 degrees
- moved IC6 111.8 mm to (103.4, 84.8), turned to 180 degrees
- moved C26 110.4 mm to (122.5, 32.0), turned to 180 degrees
- moved C25 106.9 mm to (122.5, 35.0), turned to 180 degrees
- moved C24 103.5 mm to (122.5, 38.0), turned to 180 degrees
- moved C23 100.5 mm to (122.5, 41.0), turned to 180 degrees
- moved U1 74.6 mm to (153.8, 46.7)
- moved R1 69.5 mm to (131.8, 25.2), turned to 180 degrees
- moved C3 68.8 mm to (133.5, 19.5), turned to 180 degrees
- moved R11 65.7 mm to (133.0, 45.5), turned to 180 degrees
- moved R10 65.4 mm to (133.0, 48.5), turned to 180 degrees
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Connections:
- C23 pad 1: /Sensors/SENSOR_SDA -> /Microcontroller/PERI_SDA
- C24 pad 1: /Sensors/SENSOR_SCL -> /Microcontroller/PERI_SCL
- C25 pad 1: /Sensors/LTR_INT -> /Microcontroller/LTR_INT
- IC5 pad 1: (no net) -> /Microcontroller/BAT_~{CE}
- IC5 pad 10: (no net) -> /Power/ISET
- IC5 pad 11: (no net) -> /Power/BAT+
- IC5 pad 12: (no net) -> /Power/BAT+
- IC5 pad 13: (no net) -> VBAT
- IC5 pad 14: (no net) -> VBAT
- IC5 pad 15: (no net) -> GND
- IC5 pad 16: (no net) -> GND
- IC5 pad 17: (no net) -> /Power/SW
- IC5 pad 18: (no net) -> /Power/SW
- IC5 pad 2: (no net) -> /Microcontroller/BAT_EN1
- IC5 pad 21: (no net) -> /Power/BOOT
- IC5 pad 22: (no net) -> GND
- IC5 pad 23: (no net) -> GND
- IC5 pad 24: (no net) -> /Power/LDO
- IC5 pad 25: (no net) -> GND
- IC5 pad 3: (no net) -> /Microcontroller/BAT_EN2
- IC5 pad 4: (no net) -> GND
- IC5 pad 5: (no net) -> /Input/USB_HPI_SDA
- IC5 pad 6: (no net) -> /Input/USB_HPI_SCL
- IC5 pad 7: (no net) -> /Power/STAT
- IC5 pad 8: (no net) -> /Microcontroller/BAT_INT
- IC5 pad 9: (no net) -> /Power/TS
- R18 pad 1: /Input/UART_VDD -> +3.3V
- R19 pad 1: /Input/UART_VDD -> +3.3V
- R7 pad 1: /Input/UART_VDD -> +3.3V
- U1 pad 10: unconnected-(U1-IO17-Pad10) -> /Microcontroller/S3_IO17
- U1 pad 11: unconnected-(U1-IO18-Pad11) -> /Microcontroller/S3_IO18
- U1 pad 12: unconnected-(U1-IO8-Pad12) -> /Microcontroller/LCD_EN
- U1 pad 15: unconnected-(U1-IO3-Pad15) -> /Microcontroller/S3_IO3
- U1 pad 16: unconnected-(U1-IO46-Pad16) -> /Microcontroller/S3_IO46
- U1 pad 17: unconnected-(U1-IO9-Pad17) -> /Microcontroller/S3_IO9
- U1 pad 18: unconnected-(U1-IO10-Pad18) -> /Microcontroller/S3_IO10
- U1 pad 19: unconnected-(U1-IO11-Pad19) -> /Microcontroller/S3_IO11
- U1 pad 20: unconnected-(U1-IO12-Pad20) -> /Input/USB_HPI_SDA
- U1 pad 21: unconnected-(U1-IO13-Pad21) -> /Input/USB_HPI_SCL
- U1 pad 22: unconnected-(U1-IO14-Pad22) -> /Microcontroller/S3_IO14
- U1 pad 23: unconnected-(U1-IO21-Pad23) -> /Microcontroller/S3_IO21
- U1 pad 24: unconnected-(U1-IO47-Pad24) -> /Input/USB_HPI_INT
- U1 pad 25: unconnected-(U1-IO48-Pad25) -> /Input/USB_GPIO
- U1 pad 26: unconnected-(U1-IO45-Pad26) -> /Microcontroller/S3_IO45
- U1 pad 28: unconnected-(U1-IO35-Pad28) -> /Microcontroller/S3_IO35
- U1 pad 29: unconnected-(U1-IO36-Pad29) -> /Microcontroller/S3_IO36
- U1 pad 30: unconnected-(U1-IO37-Pad30) -> /Microcontroller/S3_IO37
- U1 pad 31: unconnected-(U1-IO38-Pad31) -> /Microcontroller/S3_IO38
- U1 pad 32: unconnected-(U1-IO39-Pad32) -> /Microcontroller/BAT_EN2
- U1 pad 33: unconnected-(U1-IO40-Pad33) -> /Microcontroller/BAT_EN1
- U1 pad 34: unconnected-(U1-IO41-Pad34) -> /Microcontroller/BAT_~{CE}
- U1 pad 35: unconnected-(U1-IO42-Pad35) -> /Microcontroller/BAT_INT
- U1 pad 38: unconnected-(U1-IO2-Pad38) -> /Microcontroller/S3_IO2
- U1 pad 39: unconnected-(U1-IO1-Pad39) -> /Microcontroller/S3_IO1
- U1 pad 4: unconnected-(U1-IO4-Pad4) -> /Microcontroller/PERI_SDA
- U1 pad 5: unconnected-(U1-IO5-Pad5) -> /Microcontroller/PERI_SCL
- U1 pad 6: unconnected-(U1-IO6-Pad6) -> /Microcontroller/SOIL_EN
- U1 pad 7: unconnected-(U1-IO7-Pad7) -> /Microcontroller/SOIL_SENSE
- U1 pad 8: unconnected-(U1-IO15-Pad8) -> /Microcontroller/LTR_INT
- U1 pad 9: unconnected-(U1-IO16-Pad9) -> /Microcontroller/S3_IO16
- U5 pad 3: /Sensors/SENSOR_SDA -> /Peripherals/SENSOR_SDA
- U5 pad 4: /Sensors/SENSOR_SCL -> /Peripherals/SENSOR_SCL
- U7 pad 4: /Sensors/SENSOR_SCL -> /Microcontroller/PERI_SCL
- U7 pad 5: /Sensors/LTR_INT -> /Microcontroller/LTR_INT
- U7 pad 6: /Sensors/SENSOR_SDA -> /Microcontroller/PERI_SDA
Routing:
- net GND: track 10.3 -> 33.1 mm, vias 31 -> 39
- net VUART: track 0.00 -> 19.9 mm
- net /Input/USB_VDD: track 0.00 -> 15.4 mm
- net /Input/USB_CC2: track 2.84 -> 10.0 mm, vias 1 -> 2
- net /Input/USB_D-: track 7.73 -> 14.5 mm
- net +3.3V: track 0.00 -> 6.25 mm, vias 0 -> 1
- net /Input/USB_CC1: track 2.84 -> 8.08 mm, vias 1 -> 2
- net VUSB: track 0.00 -> 4.83 mm
- net /Input/USB_D+: track 7.18 -> 11.4 mm
- net /Input/USB_UART_D-: track 6.64 -> 9.82 mm, vias 0 -> 1
- net Net-(U4-~{RST}): track 0.35 -> 3.01 mm
- net /Input/USB_UART_D+: track 6.76 -> 8.91 mm, vias 2 -> 1
- net /Input/~{SUSPEND}: track 0.00 -> 1.82 mm, vias 0 -> 1
- net Net-(D6-A): track 0.00 -> 1.73 mm, vias 0 -> 1
- net Net-(D9-A): track 0.00 -> 1.65 mm, vias 0 -> 1
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- added copper zone on In2.Cu, net +3.3V
- added copper zone on B.Cu, net VUART
- removed copper zone on In2.Cu, net GND

Commit message: pre demo
Parts:
- removed R24: 5.1k, Resistor_SMD:R_0805_2012Metric
- removed SW1, SW3: SW_MEC_5E, AA_Switches:18259106
- removed Suspended: Yellow, LED_SMD:LED_0805_2012Metric
- added BOOT: SW_MEC_5E, AA_Switches:18259106, F.Cu at (123.0, 64.2)
- added RESET: SW_MEC_5E, AA_Switches:18259106, F.Cu at (112.0, 64.2)
- added Suspend: Yellow, LED_SMD:LED_0805_2012Metric, F.Cu at (73.2, 103.8)
- Q7, R20: moved to B.Cu
- moved J4 79.9 mm to (81.3, 35.0)
- moved Q7 78.9 mm to (82.5, 40.0), turned to 90 degrees
- moved C28 61.6 mm to (52.1, 23.2)
- moved C27 58.4 mm to (56.1, 23.2), turned to 0 degrees
- moved J2 52.9 mm to (138.8, 36.3), turned to 0 degrees
- moved C24 52.4 mm to (73.3, 19.9), turned to 90 degrees
- moved C23 52.4 mm to (72.3, 26.1), turned to -90 degrees
- moved U5 51.3 mm to (54.1, 26.0)
- moved C25 48.8 mm to (74.6, 26.1), turned to -90 degrees
- moved C26 46.6 mm to (76.8, 22.9), turned to 90 degrees
- moved J3 45.2 mm to (138.8, 40.5), turned to 0 degrees
- moved U7 39.5 mm to (74.2, 23.0)
- moved J5 37.8 mm to (138.8, 44.7), turned to 0 degrees
- moved J6 36.7 mm to (147.0, 44.5)
- moved U1 33.0 mm to (120.8, 46.1)
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- renumbered D12 to Fault
Connections:
- Recieve pad 1: /Input/TXT -> /Input/RXT
- Recieve pad 2: Net-(D9-A) -> Net-(D8-A)
- Transmit pad 1: /Input/RXT -> /Input/TXT
- Transmit pad 2: Net-(D8-A) -> Net-(D9-A)
- U5 pad 3: /Peripherals/SENSOR_SDA -> /Microcontroller/PERI_SDA
- U5 pad 4: /Peripherals/SENSOR_SCL -> /Microcontroller/PERI_SCL
Routing:
- net GND: track 33.1 -> 63.5 mm, vias 39 -> 623
- net /Microcontroller/S3_BOOT: track 0.00 -> 25.9 mm
- net /Microcontroller/PERI_SCL: track 0.00 -> 25.2 mm
- net /Microcontroller/PERI_SDA: track 0.00 -> 23.4 mm
- net /Input/USB_HPI_SCL: track 0.00 -> 22.2 mm
- net /Microcontroller/S3_EN_RST: track 0.00 -> 21.1 mm
- net /Input/USB_HPI_SDA: track 0.00 -> 20.1 mm
- net /Input/USB_FAULT: track 0.00 -> 17.2 mm, vias 0 -> 1
- net /Input/USB_D-: track 14.5 -> 24.5 mm
- net /Input/USB_D+: track 11.4 -> 21.4 mm
- net +3.3V: track 6.25 -> 16.2 mm, vias 1 -> 4
- net /Peripherals/LCD_PWR: track 0.00 -> 4.83 mm
- net /Microcontroller/LTR_INT: track 0.00 -> 4.00 mm
- net VUSB: track 4.83 -> 7.83 mm
- net /Input/USB_GPIO: track 0.00 -> 2.39 mm
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- added copper zone on B.Cu, net GND
Other:
- board outline added: 100.5 x 100.5 mm
- board text added: "H1"
