File: GreenNet/GreenNet.kicad_pcb (KiCad board)
At the start: 4 copper layers, 100.5 x 100.5 mm, 110 parts, among them IC5 BQ24250RGER, IC6 NCP186AMX330TAG, J1 Conn_01x03_Pin, J2 3_Pin_Conn, J3 3_Pin_Conn, J4 Conn_01x04_Pin, J5 3_Pin_Conn, J6 Conn_01x14_Pin, Q3 IRF9358TRPBF, Q4 SI3932DV-T1-GE3, Q5 SI3993CDV-T1-GE3, Q6 2N7002K, Q7 2N7002K, Q8 MMDT3904, U1 ESP32-S3-WROOM-1-N16R2, U2 USB_C_Receptacle_12P, U3 USB_C_Receptacle_12P, U4 CP2102N-A02-GQFN28, U5 BME280, U6 CYPD3177-24LQXQT, U7 LTR-303ALS-01

Commit message: schematic FINAL
Parts:
- removed BOOT, RESET: SW_MEC_5E, AA_Switches:18259106
- removed Suspend: Yellow, LED_SMD:LED_0805_2012Metric
- added R24: 5.1k, Resistor_SMD:R_0805_2012Metric, F.Cu at (103.6, 62.5)
- added SW1: SW_MEC_5E, AA_Switches:18259106, F.Cu at (136.2, 76.2)
- added SW3: SW_MEC_5E, AA_Switches:18259106, F.Cu at (136.2, 67.1)
- added Suspended: Yellow, LED_SMD:LED_0805_2012Metric, F.Cu at (73.2, 103.8)
- Q7, R20: moved to F.Cu
- moved J4 79.9 mm to (142.5, 86.2)
- moved Q7 78.9 mm to (142.1, 91.7), turned to 180 degrees
- moved C28 61.6 mm to (112.7, 34.7)
- moved C27 58.4 mm to (112.7, 37.7), turned to 180 degrees
- moved J2 52.9 mm to (158.8, 85.2), turned to 180 degrees
- moved C24 52.4 mm to (122.5, 38.0), turned to 180 degrees
- moved C23 52.4 mm to (122.5, 41.0), turned to 180 degrees
- moved U5 51.3 mm to (103.3, 40.5)
- moved C25 48.8 mm to (122.5, 35.0), turned to 180 degrees
- moved C26 46.6 mm to (122.5, 32.0), turned to 180 degrees
- moved J3 45.2 mm to (158.8, 81.0), turned to 180 degrees
- moved U7 39.5 mm to (113.4, 27.8)
- moved J5 37.8 mm to (158.8, 76.8), turned to 180 degrees
- moved J6 36.7 mm to (166.0, 75.9)
- moved U1 33.0 mm to (153.8, 46.7)
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- renumbered Fault to D12
Connections:
- Recieve pad 1: /Input/RXT -> /Input/TXT
- Recieve pad 2: Net-(D8-A) -> Net-(D9-A)
- Transmit pad 1: /Input/TXT -> /Input/RXT
- Transmit pad 2: Net-(D9-A) -> Net-(D8-A)
- U5 pad 3: /Microcontroller/PERI_SDA -> /Peripherals/SENSOR_SDA
- U5 pad 4: /Microcontroller/PERI_SCL -> /Peripherals/SENSOR_SCL
Routing:
- net GND: track 63.5 -> 33.1 mm, vias 623 -> 39
- net /Microcontroller/S3_BOOT: track 25.9 -> 0.00 mm
- net /Microcontroller/PERI_SCL: track 25.2 -> 0.00 mm
- net /Microcontroller/PERI_SDA: track 23.4 -> 0.00 mm
- net /Input/USB_HPI_SCL: track 22.2 -> 0.00 mm
- net /Microcontroller/S3_EN_RST: track 21.1 -> 0.00 mm
- net /Input/USB_HPI_SDA: track 20.1 -> 0.00 mm
- net /Input/USB_FAULT: track 17.2 -> 0.00 mm, vias 1 -> 0
- net /Input/USB_D-: track 24.5 -> 14.5 mm
- net /Input/USB_D+: track 21.4 -> 11.4 mm
- net +3.3V: track 16.2 -> 6.25 mm, vias 4 -> 1
- net /Peripherals/LCD_PWR: track 4.83 -> 0.00 mm
- net /Microcontroller/LTR_INT: track 4.00 -> 0.00 mm
- net VUSB: track 7.83 -> 4.83 mm
- net /Input/USB_GPIO: track 2.39 -> 0.00 mm
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- removed copper zone on B.Cu, net GND
Other:
- board outline removed
- board text removed: "H1"

Commit message: layout update
Parts:
- removed BT1: Battery_Cell, AA_Connectors:BH18650PC
- removed C21: 2.2u, Capacitor_SMD:C_0805_2012Metric
- removed C22, C26, C31, C32: 1u, Capacitor_SMD:C_0805_2012Metric
- removed C23, C24, C25: 10p, Capacitor_SMD:C_0805_2012Metric
- removed C27, C28: 0.1u, Capacitor_SMD:C_0805_2012Metric
- removed C29: 33n, Capacitor_SMD:C_0805_2012Metric
- removed C30: 22u, Capacitor_SMD:C_0805_2012Metric
- removed Connected (x2), Recieve, Transmit: Green, LED_SMD:LED_0805_2012Metric
- removed D14, D15: D5V0M1U2S9, AA_Diodes:D5V0M1U2S9Q
- removed IC5: BQ24250RGER, QFN:QFN50P400X400X100-25N-D
- removed IC6: NCP186AMX330TAG, AA_Power_ICs:NCP186AMX330TAG
- removed J6: Conn_01x14_Pin, AA_Connectors:CONN_PH1-14-UA_ADM
- removed Q3: IRF9358TRPBF, AA_FETS:SO8_IRF9358TRPBF_INF
- removed Q4: SI3932DV-T1-GE3, AA_FETS:TSOP_0DV-T1-E3_VIS
- removed Q5: SI3993CDV-T1-GE3, AA_FETS:TSOP_0DV-T1-E3_VIS
- removed Q6, Q7: 2N7002K, Package_TO_SOT_SMD:SOT-23
- removed Q8: MMDT3904, Package_TO_SOT_SMD:SOT-363_SC-70-6
- removed R19, R20, R7, R8: 62R, Resistor_SMD:R_0805_2012Metric
- removed R21: 12k, Resistor_SMD:R_0805_2012Metric
- removed R22, R24: 5.1k, Resistor_SMD:R_0805_2012Metric
- removed R23, R6: 1k, Resistor_SMD:R_0805_2012Metric
- removed R25: 2.4k, Resistor_SMD:R_0805_2012Metric
- removed R26: 1.3k, Resistor_SMD:R_0805_2012Metric
- removed R27: 150R, Resistor_SMD:R_0805_2012Metric
- removed R28, R29, R30, R31, R32, R33, R34: 10k, Resistor_SMD:R_0805_2012Metric
- removed SW3: SW_MEC_5E, AA_Switches:18259106
- removed Suspended: Yellow, LED_SMD:LED_0805_2012Metric
- removed TH1: R_{0}= 10K, B = 3470K, AA_Resistors:MF52A2103J3470
- added D11: DSS14U, AA_Diodes:DSS14U, F.Cu at (82.0, 71.4)
- added D5: D5V0M1U2S9, AA_Diodes:D5V0M1U2S9Q, F.Cu at (80.2, 76.7)
- added D6: D5V0M1U2S9, AA_Diodes:D5V0M1U2S9Q, F.Cu at (80.2, 63.2)
- added D8: D5V0M1U2S9, AA_Diodes:D5V0M1U2S9Q, F.Cu at (78.5, 65.8)
- added D9: D5V0M1U2S9, AA_Diodes:D5V0M1U2S9Q, F.Cu at (78.2, 76.4)
- added Q1: MMDT3904, Package_TO_SOT_SMD:SOT-363_SC-70-6, F.Cu at (239.8, 91.9)
- added Q2: 2N7002K, Package_TO_SOT_SMD:SOT-23, F.Cu at (215.1, 126.6)
- added SW2: SW_MEC_5E, AA_Switches:18259106, F.Cu at (228.9, 89.3)
- added TP1: TestPoint, AA_TestPoints:RCWCTE, F.Cu at (238.8, 97.7)
- added TP10: TestPoint, AA_TestPoints:RCWCTE, F.Cu at (196.4, 128.2)
- added TP11: TestPoint, AA_TestPoints:RCWCTE, F.Cu at (196.4, 131.3)
- added TP12: TestPoint, AA_TestPoints:RCWCTE, F.Cu at (196.4, 134.5)
- added TP13: SOIL_SENSE, AA_TestPoints:RCWCTE, F.Cu at (196.4, 137.6)
- added TP2: TestPoint, AA_TestPoints:RCWCTE, F.Cu at (238.8, 100.9)
- added TP3: TestPoint, AA_TestPoints:RCWCTE, F.Cu at (238.8, 104.0)
- added TP4: TestPoint, AA_TestPoints:RCWCTE, F.Cu at (238.8, 107.2)
- added TP5: TestPoint, AA_TestPoints:RCWCTE, F.Cu at (196.4, 112.4)
- added TP6: TestPoint, AA_TestPoints:RCWCTE, F.Cu at (196.4, 115.6)
- added TP7: VBUS, AA_TestPoints:RCWCTE, F.Cu at (196.4, 118.7)
- added TP8: SOIL_EN, AA_TestPoints:RCWCTE, F.Cu at (196.4, 121.9)
- added TP9: TestPoint, AA_TestPoints:RCWCTE, F.Cu at (196.4, 125.0)
- C1: value 10u -> 1u
- C10: value 10u -> 22u; moved to F.Cu
- C11: value 1u -> 22u
- C13, C19: moved to B.Cu
- C14: value 0.1u -> 10p
- C15: value 390p -> 4.7u
- C16: value 390p -> 10p; moved to F.Cu
- C17: value 1u -> 0.1u; moved to B.Cu
- C18: value 1u -> 10p
- C2, C4: value 0.1u -> 10u
- C20: value 1u -> 10u; moved to B.Cu
- C3: value 1u -> 0.1u
- C5: value 4.7u -> 10u
- C6: value 0.1u -> 10u; moved to F.Cu
- C7: value 1u -> 0.1u; moved to F.Cu
- C8, C9: value 10u -> 0.1u; moved to F.Cu
- D10: value D5V0M1U2S9 -> DSS14U; footprint AA_Diodes:D5V0M1U2S9Q -> AA_Diodes:DSS14U
- D12: value Red -> Green
- D13: value Yellow -> Green
- D3: value D5V0M1U2S9 -> Green; footprint AA_Diodes:D5V0M1U2S9Q -> LED_SMD:LED_0805_2012Metric
- D4: moved to F.Cu
- D7: value 10V -> D5V0M1U2S9; footprint AA_Diodes:NHZ10C,115 -> AA_Diodes:D5V0M1U2S9Q
- J1: value Conn_01x03_Pin -> 3_Pin_Conn
- J4: value Conn_01x04_Pin -> Conn_01x20_Pin; footprint AA_Connectors:61300411121 -> AA_Connectors:CONN_PH2-20-UA_ADM
- J5: value 3_Pin_Conn -> Conn_01x03_Pin
- L1: value 1u -> 3.9u; footprint Inductor_SMD:L_0805_2012Metric -> AA_Inductors:ASPI0628150MT1
- R11: value 10k -> 62R
- R12, R14: value 49.9k -> 5.1k; moved to B.Cu
- R13: value 1k -> 5.1k; moved to B.Cu
- R15: value 62R -> 5.1k
- R16: value 49.9k -> 150R; moved to B.Cu
- R17: value 5.6k -> 150R; moved to B.Cu
- R18: value 62R -> 1k; moved to F.Cu
- R2, R9: value 1k -> 10k
- R4, R5: value 5.1k -> 10k; moved to F.Cu
- U1: value ESP32-S3-WROOM-1-N16R2 -> ESP32-S3-WROOM-1-N4R2
- U4: value CP2102N-A02-GQFN28 -> AP63203WU; footprint Package_DFN_QFN:QFN-28-1EP_5x5mm_P0.5mm_EP3.35x3.35mm -> Package_TO_SOT_SMD:TSOT-23-6; moved to F.Cu
- U6: value CYPD3177-24LQXQT -> CP2102N-A02-GQFN28; footprint AA_Interface_USB:QFN50P400X400X60-25N-D -> Package_DFN_QFN:QFN-28-1EP_5x5mm_P0.5mm_EP3.35x3.35mm
- moved H2 166.7 mm to (218.9, 87.7)
- moved H3 166.7 mm to (218.9, 94.2)
- moved H4 166.7 mm to (218.9, 100.8)
- moved D3 160.3 mm to (240.0, 88.4), turned to 0 degrees
- moved H1 153.5 mm to (218.9, 81.1)
- moved R4 152.7 mm to (224.4, 88.2)
- moved R5 152.3 mm to (224.4, 91.1)
- moved U7 144.9 mm to (195.5, 147.2), turned to 0 degrees
- moved D1 144.9 mm to (223.6, 102.5), turned to 0 degrees
- moved U5 144.8 mm to (219.8, 126.5), turned to 0 degrees
- moved D2 144.1 mm to (223.6, 104.5), turned to 0 degrees
- moved C16 140.7 mm to (210.4, 112.4), turned to 0 degrees
- moved R9 132.0 mm to (224.4, 94.1), turned to 0 degrees
- moved R3 130.4 mm to (224.4, 85.2), turned to 0 degrees
- moved C8 126.5 mm to (201.5, 124.4), turned to 0 degrees
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Connections:
- C1 pad 1: +3.3V -> /Microcontroller/S3_EN_RST
- C10 pad 1: VUSB -> +3.3V
- C11 pad 1: /Input/FET_GATE -> +3.3V
- C11 pad 2: VUSB -> GND
- C12 pad 1: /Input/FET_GATE -> +3.3V
- C12 pad 2: VBUS -> GND
- C13 pad 1: /Input/USB_VDD -> /Input/UART_VDD
- C14 pad 1: /Input/USB_VDD -> /Input/PERI_SDA
- C15 pad 1: /Input/USB_CC1 -> /Input/UART_VDD
- C16 pad 1: /Input/USB_CC2 -> /Input/PERI_SCL
- C17 pad 1: /Input/USB_VCC -> VUART
- C18 pad 1: /Input/USB_VDD -> /Input/LTR_INT
- C19 pad 1: +3.3V -> VUART
- C20 pad 1: VBAT -> VUART
- C3 pad 1: /Microcontroller/S3_EN_RST -> +3.3V
- C4 pad 1: /Input/UART_VDD -> VUSB
- C5 pad 1: /Input/UART_VDD -> VUART
- C6 pad 1: VUART -> VBUS
- C7 pad 1: VUART -> +3.3V
- C8 pad 1: VUART -> +3.3V
- C9 pad 1: VUART -> Net-(U4-SW)
- C9 pad 2: GND -> Net-(U4-BST)
- D1 pad 1: /Input/USB_D+ -> /Microcontroller/S3_BOOT
- D10 pad 1: /Input/USB_D- -> VBUS
- D10 pad 2: GND -> VUSB
- D13 pad 1: /Power/STAT -> GND
- D2 pad 1: /Input/USB_UART_D+ -> /Microcontroller/S3_EN_RST
- D3 pad 1: /Input/USB_UART_D- -> GND
- D3 pad 2: GND -> Net-(D3-A)
- D4 pad 1: VUART -> /Input/USB_D+
- D7 pad 1: /Input/FET_SRC -> /Input/USB_UART_D-
- D7 pad 2: /Input/FET_GATE -> GND
- J1 pad 1: /Microcontroller/SOIL_SENSE -> +3.3V
- J1 pad 2: /Peripherals/SOIL_PWR -> /Microcontroller/S3_IO3
- J2 pad 2: /Microcontroller/S3_IO3 -> /Microcontroller/S3_IO45
- J3 pad 2: /Microcontroller/S3_IO45 -> /Microcontroller/S3_IO46
- J4 pad 1: /Microcontroller/PERI_SCL -> /Microcontroller/S3_IO1
- J4 pad 2: /Microcontroller/PERI_SDA -> /Microcontroller/S3_IO2
- J4 pad 3: /Peripherals/LCD_PWR -> /Microcontroller/S3_IO9
- J4 pad 4: GND -> /Microcontroller/S3_IO10
- J5 pad 1: +3.3V -> /Input/SOIL_SENSE
- J5 pad 2: /Microcontroller/S3_IO46 -> /Input/SOIL_PWR
- L1 pad 1: /Power/SW -> Net-(U4-SW)
- L1 pad 2: VBAT -> +3.3V
- R1 pad 1: /Microcontroller/S3_EN_RST -> /Microcontroller/PWR_SDA
- R10 pad 1: /Input/UART_~{RTS} -> /Input/UART_~{DTR}
- R11 pad 1: /Input/UART_~{DTR} -> /Microcontroller/LED_TEST
- R11 pad 2: Net-(Q8A-B1) -> Net-(D3-A)
- R12 pad 1: /Input/FET_GATE -> GND
- R12 pad 2: /Input/FET_SRC -> Net-(U2-CC2)
- R13 pad 1: Net-(Q5-G1) -> GND
- R13 pad 2: /Input/SAFE_PWR_EN -> Net-(U3-CC2)
- R14 pad 1: Net-(Q5-G1) -> GND
- R14 pad 2: VUSB -> Net-(U2-CC1)
- R15 pad 1: /Input/USB_VDD -> GND
- R15 pad 2: Net-(D11-A) -> Net-(U3-CC1)
- R16 pad 1: GND -> VUSB
- R16 pad 2: Net-(Q4-G1) -> Net-(D12-A)
- R17 pad 1: /Power/LDO -> VUART
- R17 pad 2: /Power/TS -> Net-(D13-A)
- R18 pad 1: +3.3V -> /Input/UART_VDD
- R18 pad 2: Net-(D9-A) -> Net-(U6-~{RST})
- R2 pad 1: Net-(Q4-G1) -> /Microcontroller/S3_EN_RST
- R2 pad 2: /Input/UART_VDD -> +3.3V
- R3 pad 1: /Input/FET_GATE -> /Microcontroller/PWR_SCL
- R3 pad 2: VUSB -> +3.3V
- R4 pad 1: GND -> /Input/PERI_SDA
- R4 pad 2: Net-(U3-CC2) -> +3.3V
- R5 pad 1: GND -> /Input/PERI_SCL
- R5 pad 2: Net-(U3-CC1) -> +3.3V
- R9 pad 1: /Input/FET_GATE -> /Input/UART_~{RTS}
- R9 pad 2: /Input/VBUS_FET_EN -> Net-(Q1B-B2)
- SW1 pad 1: /Microcontroller/S3_EN_RST -> /Microcontroller/S3_BOOT
- SW1 pad 2: /Microcontroller/S3_EN_RST -> /Microcontroller/S3_BOOT
- U1 pad 12: /Microcontroller/LCD_EN -> /Microcontroller/LED_TEST
- U1 pad 20: /Input/USB_HPI_SDA -> /Microcontroller/PWR_SDA
- U1 pad 21: /Input/USB_HPI_SCL -> /Microcontroller/PWR_SCL
- U1 pad 24: /Input/USB_HPI_INT -> /Microcontroller/S3_IO47
- U1 pad 25: /Input/USB_GPIO -> /Microcontroller/S3_IO48
- U1 pad 32: /Microcontroller/BAT_EN2 -> /Microcontroller/S3_IO39
- U1 pad 33: /Microcontroller/BAT_EN1 -> /Microcontroller/S3_IO40
- U1 pad 34: /Microcontroller/BAT_~{CE} -> /Microcontroller/S3_IO41
- U1 pad 35: /Microcontroller/BAT_INT -> /Microcontroller/S3_IO42
- U1 pad 4: /Microcontroller/PERI_SDA -> /Input/PERI_SDA
- U1 pad 5: /Microcontroller/PERI_SCL -> /Input/PERI_SCL
- U1 pad 6: /Microcontroller/SOIL_EN -> /Input/SOIL_EN
- U1 pad 7: /Microcontroller/SOIL_SENSE -> /Input/SOIL_SENSE
- U1 pad 8: /Microcontroller/LTR_INT -> /Input/LTR_INT
- U2 pad A5: /Input/USB_CC1 -> Net-(U2-CC1)
- U2 pad B5: /Input/USB_CC2 -> Net-(U2-CC2)
- U4 pad 1: unconnected-(U4-~{DCD}-Pad1) -> +3.3V
- U4 pad 2: unconnected-(U4-~{RI}/CLK-Pad2) -> VBUS
- U4 pad 3: GND -> VBUS
- U4 pad 4: /Input/USB_UART_D+ -> GND
- U4 pad 5: /Input/USB_UART_D- -> Net-(U4-SW)
- U4 pad 6: /Input/UART_VDD -> Net-(U4-BST)
- U5 pad 3: /Peripherals/SENSOR_SDA -> /Input/PERI_SDA
- U5 pad 4: /Peripherals/SENSOR_SCL -> /Input/PERI_SCL
- U6 pad 1: GND -> unconnected-(U6-~{DCD}-Pad1)
- U6 pad 11: VBUS -> unconnected-(U6-~{SUSPEND}-Pad11)
- U6 pad 12: /Input/USB_HPI_SDA -> unconnected-(U6-SUSPEND-Pad12)
- U6 pad 13: /Input/USB_HPI_SCL -> unconnected-(U6-CHREN-Pad13)
- U6 pad 14: /Input/USB_CC2 -> unconnected-(U6-CHR1-Pad14)
- U6 pad 15: /Input/USB_CC1 -> unconnected-(U6-CHR0-Pad15)
- U6 pad 18: VUSB -> unconnected-(U6-RXT-Pad18)
- U6 pad 19: GND -> unconnected-(U6-TXT-Pad19)
- U6 pad 2: /Input/VBUS_MAX -> unconnected-(U6-~{RI}/CLK-Pad2)
- U6 pad 22: GND -> unconnected-(U6-GPIO.4-Pad22)
- U6 pad 23: /Input/USB_VDD -> unconnected-(U6-~{CTS}-Pad23)
- U6 pad 24: /Input/USB_VCC -> /Input/UART_~{RTS}
- U6 pad 25: GND -> /Input/UART_RXD
- U6 pad 3: /Input/VBUS_FET_EN -> GND
- U6 pad 4: /Input/SAFE_PWR_EN -> /Input/USB_UART_D+
- U6 pad 5: /Input/ISNK_COARSE -> /Input/USB_UART_D-
- U6 pad 6: GND -> /Input/UART_VDD
- U6 pad 7: /Input/USB_HPI_INT -> VUART
- U6 pad 8: /Input/USB_GPIO -> VUART
- U6 pad 9: /Input/USB_FAULT -> Net-(U6-~{RST})
- U7 pad 4: /Microcontroller/PERI_SCL -> /Input/PERI_SCL
- U7 pad 5: /Microcontroller/LTR_INT -> /Input/LTR_INT
- U7 pad 6: /Microcontroller/PERI_SDA -> /Input/PERI_SDA
Routing:
- net GND: track 33.1 -> 9.62 mm, vias 39 -> 392
- net /Input/USB_VDD: track 15.4 -> 0.00 mm
- net /Input/USB_D-: track 14.5 -> 3.81 mm
- net /Input/USB_CC2: track 10.0 -> 0.00 mm, vias 2 -> 0
- net Net-(U4-SW): track 0.00 -> 9.83 mm
- net /Input/USB_D+: track 11.4 -> 3.32 mm
- net /Input/USB_CC1: track 8.08 -> 0.00 mm, vias 2 -> 0
- net VBUS: track 0.00 -> 5.95 mm
- net +3.3V: track 6.25 -> 11.9 mm
- net VUSB: track 4.83 -> 10.0 mm, vias 16 -> 24
- net Net-(U4-~{RST}): track 3.01 -> 0.00 mm
- net Net-(U6-~{RST}): track 0.00 -> 2.68 mm, vias 0 -> 1
- net Net-(U2-CC2): track 0.00 -> 2.38 mm, vias 0 -> 1
- net Net-(U2-CC1): track 0.00 -> 2.28 mm, vias 0 -> 1
- net /Input/~{SUSPEND}: track 1.82 -> 0.00 mm, vias 1 -> 0
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- added copper zone on F.Cu, net +3.3V
- removed copper zone on F.Cu, net GND
- removed copper zone on In1.Cu, net VUSB
Other:
- board outline added: 100 x 100 mm

Commit message: update
Parts:
- removed R1: 10k, Resistor_SMD:R_0805_2012Metric
- added H5: MountingHole_Pad, MountingHole:MountingHole_2.5mm_Pad, F.Cu at (107.2, 37.0)
- C18, TP1, TP10, TP11, TP12, TP13, TP2, TP5, TP6, TP8, TP9: moved to B.Cu
- moved J5 163.8 mm to (72.0, 46.5), turned to 90 degrees
- moved Q2 160.5 mm to (76.0, 46.5), turned to 180 degrees
- moved H2 154.9 mm to (72.5, 37.0)
- moved TP1 152.5 mm to (94.8, 47.8)
- moved TP13 150.3 mm to (72.0, 53.2), turned to -90 degrees
- moved TP2 150.2 mm to (97.5, 50.0)
- moved U7 148.1 mm to (89.3, 43.9), turned to -90 degrees
- moved H3 146.4 mm to (72.5, 96.0)
- moved U5 144.6 mm to (99.8, 45.9), turned to -90 degrees
- moved C18 142.4 mm to (87.2, 47.0), turned to 180 degrees
- moved C16 141.3 mm to (86.7, 44.0), turned to 90 degrees
- moved C12 139.8 mm to (89.5, 41.0), turned to 180 degrees
- moved C14 139.5 mm to (92.0, 44.0), turned to 90 degrees
- moved TP8 137.9 mm to (80.5, 47.2), turned to -90 degrees
- moved C2 137.1 mm to (107.0, 48.8), turned to 90 degrees
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Connections:
- R3 pad 1: /Microcontroller/PWR_SCL -> /Input/LTR_INT
- U1 pad 20: /Microcontroller/PWR_SDA -> unconnected-(U1-IO12-Pad20)
- U1 pad 21: /Microcontroller/PWR_SCL -> unconnected-(U1-IO13-Pad21)
Routing:
- net /Input/UART_TXD: track 0.00 -> 73.9 mm, vias 0 -> 1
- net /Input/UART_RXD: track 0.00 -> 72.2 mm, vias 0 -> 1
- net /Microcontroller/S3_IO14: track 0.00 -> 51.7 mm, vias 0 -> 1
- net /Input/SOIL_SENSE: track 0.00 -> 50.6 mm
- net /Input/PERI_SCL: track 0.00 -> 49.4 mm, vias 0 -> 4
- net /Input/SOIL_EN: track 0.00 -> 49.0 mm, vias 0 -> 1
- net /Microcontroller/S3_EN_RST: track 0.00 -> 48.2 mm, vias 0 -> 1
- net /Input/USB_D-: track 3.81 -> 51.6 mm, vias 0 -> 1
- net /Input/UART_~{DTR}: track 0.00 -> 46.7 mm, vias 0 -> 1
- net /Input/USB_D+: track 3.32 -> 49.1 mm, vias 0 -> 1
- net /Input/PERI_SDA: track 0.00 -> 45.7 mm, vias 0 -> 4
- net /Input/LTR_INT: track 0.00 -> 40.9 mm, vias 0 -> 2
- net /Microcontroller/S3_IO21: track 0.00 -> 39.6 mm, vias 0 -> 1
- net /Input/UART_~{RTS}: track 0.00 -> 39.6 mm, vias 0 -> 3
- net /Microcontroller/S3_IO46: track 0.00 -> 37.0 mm, vias 0 -> 1
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- added copper zone on B.Cu, net GND
- added copper zone on F.Cu, net GND
Other:
- board size 100 x 100 mm -> 84.8 x 67 mm

Commit message: update
Parts:
- TP1: value TestPoint -> PERI_SDA
- TP10: value TestPoint -> USB_D+
- TP11: value TestPoint -> USB_UART_D-
- TP12: value TestPoint -> USB_UART_D+
- TP2: value TestPoint -> PERI_SCL
- TP3: value TestPoint -> S3_EN_RST
- TP4: value TestPoint -> S3_BOOT
- TP5: value TestPoint -> UART_TXD
- TP6: value TestPoint -> UART_RXD
- TP9: value TestPoint -> USB_D-
- moved TP10 0.25 mm to (85.8, 58.8)
Routing:
- net +3.3V: track 39.6 -> 44.1 mm
- net GND: vias 471 -> 426
- removed copper zone on B.Cu, net GND
- removed copper zone on F.Cu, net GND
Other:
- board text added: "${REFERENCE}"
