File: GreenNet/peripherals.kicad_sch (KiCad schematic)
At the start: 18 parts, among them J1 Conn_01x03_Pin, J4 Conn_01x04_Pin, Q6 2N7002K, Q7 2N7002K, U5 BME280, U7 LTR-303ALS-01

Commit message: pre demo
Connections:
- net SENSOR_SCL is gone; now on net PERI_SCL: U5.4 (SCK)
- net SENSOR_SDA is gone; now on net PERI_SDA: U5.3 (SDI)
Changed lines of the file:
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@@
-		)
-	)
-	(label "SENSOR_SDA"
-		(at 60.96 62.23 180)
-		(fields_autoplaced yes)
-		(effects
-			(font
-				(size 1.27 1.27)
-			)
-			(justify right bottom)
 		)
 	)
@@
 			)
 			(justify left bottom)
+		)
+	)
+	(label "PERI_SCL"
+		(at 60.96 64.77 180)
+		(fields_autoplaced yes)
+		(effects
+			(font
+				(size 1.27 1.27)
+			)
+			(justify right bottom)
 		)
 	)
@@
 		)
 	)
-	(label "SENSOR_SCL"
-		(at 60.96 64.77 180)
-		(fields_autoplaced yes)
-		(effects
-			(font
-				(size 1.27 1.27)
-			)
-			(justify right bottom)
-		)
-	)
 	(label "PERI_SCL"
 		(at 220.98 60.96 0)
@@
 		)
 	)
+	(label "PERI_SDA"
+		(at 60.96 62.23 180)
+		(fields_autoplaced yes)
+		(effects
+			(font
+				(size 1.27 1.27)
+			)
+			(justify right bottom)
+		)
+	)
