File: GreenNet/power.kicad_sch (KiCad schematic)
At the start: 1 part, among them U5 MC33063AD

Commit message: USB-PC PD progress
Parts:
- added IC1: BQ24250RGET, QFN50P400X400X100-25N-D, symbol AA_Power_ICs:BQ24250RGET
Connections:
- new net: IC1.11 (BAT), IC1.12 (BAT)
- new net: IC1.13 (SYS), IC1.14 (SYS)
- new net: IC1.15 (PGND), IC1.16 (PGND)
- new net: IC1.17 (SW), IC1.18 (SW)
Other:
- moved on the sheet: U5
Changed lines of the file:
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@@
 	(wire
 		(pts
-			(xy 107.95 86.36) (xy 107.95 87.63)
+			(xy 163.83 99.06) (xy 163.83 100.33)
 		)
 		(stroke
@@
 	(symbol
 		(lib_id "power:GND")
-		(at 107.95 87.63 0)
+		(at 163.83 100.33 0)
 		(unit 1)
 		(exclude_from_sim no)
@@
 		(fields_autoplaced yes)
 		(property "Reference" "#PWR036"
-			(at 107.95 93.98 0)
+			(at 163.83 106.68 0)
 			(effects
 				(font
@@
 		)
 		(property "Value" "GND"
-			(at 107.95 92.71 0)
+			(at 163.83 105.41 0)
 			(effects
 				(font
@@
 		)
 		(property "Footprint" ""
-			(at 107.95 87.63 0)
+			(at 163.83 100.33 0)
 			(effects
 				(font
@@
 		)
 		(property "Datasheet" ""
-			(at 107.95 87.63 0)
+			(at 163.83 100.33 0)
 			(effects
 				(font
@@
 		)
 		(property "Description" "Power symbol creates a global label with name \"GND\" , ground"
-			(at 107.95 87.63 0)
+			(at 163.83 100.33 0)
 			(effects
 				(font
@@
 	)
 	(symbol
+		(lib_id "AA_Power_ICs:BQ24250RGET")
+		(at 109.22 86.36 0)
+		(unit 1)
+		(exclude_from_sim no)
+		(in_bom yes)
+		(on_board yes)
+		(dnp no)
+		(fields_autoplaced yes)
+		(property "Reference" "IC1"
+			(at 113.9541 68.58 0)
+			(effects
+				(font
+					(size 1.27 1.27)
+				)
+				(justify left)
+			)
+		)
+		(property "Value" "BQ24250RGET"
+			(at 113.9541 71.12 0)
+			(effects
+				(font
+					(size 1.27 1.27)
+				)
+				(justify left)
+			)
+		)
+		(property "Footprint" "QFN50P400X400X100-25N-D"
+			(at 156.464 73.406 0)
+			(effects
+				(font
+					(size 1.27 1.27)
+				)
+				(justify left top)
+				(hide yes)
+			)
+		)
+		(property "Datasheet" "https://www.ti.com/lit/ds/symlink/bq24250.pdf"
+			(at 156.464 77.724 0)
+			(effects
+				(font
+					(size 1.27 1.27)
+				)
+				(justify left top)
+				(hide yes)
+			)
+		)
+		(property "Description" "2A Single Input I2C/Standalone Switch-Mode Li-Ion Battery Charger"
+			(at 190.246 76.2 0)
+			(effects
+				(font
+					(size 1.27 1.27)
+				)
+				(hide yes)
+			)
+		)
+		(property "Height" "1"
+			(at 135.89 473.66 0)
+			(effects
+				(font
+					(size 1.27 1.27)
+				)
+				(justify left top)
+				(hide yes)
+			)
+		)
+		(property "Manufacturer_Name" "Texas Instruments"
+			(at 156.464 71.12 0)
+			(effects
+				(font
+					(size 1.27 1.27)
+				)
+				(justify left top)
+				(hide yes)
+			)
+		)
+		(pin "16"
+		)
+		(pin "12"
+		)
+		(pin "8"
+		)
+		(pin "21"
+		)
+		(pin "5"
+		)
+		(pin "10"
+		)
+		(pin "14"
+		)
+		(pin "18"
+		)
+		(pin "7"
+		)
+		(pin "2"
+		)
+		(pin "19"
+		)
+		(pin "15"
+		)
+		(pin "20"
+		)
+		(pin "13"
+		)
+		(pin "3"
+		)
+		(pin "6"
+		)
+		(pin "4"
+		)
+		(pin "1"
+		)
+		(pin "22"
+		)
+		(pin "9"
+		)
+		(pin "25"
+		)
+		(pin "11"
+		)
+		(pin "23"
+		)
+		(pin "17"
+		)
+		(pin "24"
+		)
+		(instances
+			(project ""
+				(path "/189669a5-f2fc-4cde-9413-8df80c557655/25a95746-0a87-4e99-99e5-3474e5066d9d"
+					(reference "IC1")
+					(unit 1)
+				)
+			)
+		)
+	)
+	(symbol
 		(lib_id "Regulator_Switching:MC33063AD")
-		(at 107.95 73.66 0)
+		(at 163.83 86.36 0)
 		(unit 1)
 		(exclude_from_sim no)
@@
 		(dnp no)
 		(property "Reference" "U5"
-			(at 114.554 85.09 0)
+			(at 170.434 97.79 0)
 			(effects
 				(font
@@
 		)
 		(property "Value" "MC33063AD"
-			(at 107.95 64.77 0)
+			(at 163.83 77.47 0)
 			(effects
 				(font
@@
 		)
 		(property "Footprint" "Package_SO:SOIC-8_3.9x4.9mm_P1.27mm"
-			(at 109.22 85.09 0)
+			(at 165.1 97.79 0)
 			(effects
 				(font
@@
 		)
 		(property "Datasheet" "http://www.onsemi.com/pub_link/Collateral/MC34063A-D.PDF"
-			(at 120.65 76.2 0)
+			(at 176.53 88.9 0)
 			(effects
 				(font
@@
 		)
 		(property "Description" "1.5A, step-up/down/inverting switching regulator, 3-40V Vin, 100kHz, SO-8"
-			(at 107.95 73.66 0)
-			(effects
-				(font
+			(at 163.83 86.36 0)
+			(effects
+				(font

Commit message: started layout
Parts:
- IC1: footprint QFN50P400X400X100-25N-D -> QFN:QFN50P400X400X100-25N-D
Changed lines of the file:
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@@
 			)
 		)
-		(property "Footprint" "QFN50P400X400X100-25N-D"
+		(property "Footprint" "QFN:QFN50P400X400X100-25N-D"
 			(at 156.464 73.406 0)
 			(effects

Commit message: more sensor work
Parts:
- removed IC1: BQ24250RGET, QFN:QFN50P400X400X100-25N-D, symbol AA_Power_ICs:BQ24250RGET
- removed U5: MC33063AD, Package_SO:SOIC-8_3.9x4.9mm_P1.27mm, symbol Regulator_Switching:MC33063AD
- added C19, C20: 1u, Capacitor_SMD:C_0805_2012Metric, symbol Device:C
- added IC5: BQ24250RGER, QFN50P400X400X100-25N-D, symbol AA_Power_ICs:BQ24250RGET
- added IC6: NCP186AMX330TAG, AA_Power_ICs:NCP186AMX330TAG, symbol AA_Power_ICs:NCP186AMX330TAG
Connections:
- net VBUS: now also IC5.19 (IN)
- new net: IC5.11 (BAT), IC5.12 (BAT)
- new net: IC5.13 (SYS), IC5.14 (SYS)
- new net: IC5.15 (PGND), IC5.16 (PGND), IC5.25 (EP), IC5.4 (AGND)
- new net: IC5.17 (SW), IC5.18 (SW)
- new net +3.3V: C19.1, IC6.1 (OUT), IC6.2 (OUT), IC6.4 (FB)
- new net EPAD: C19.2, C20.2, IC6.3 (NC), IC6.5 (GND), IC6.9 (EPAD)
- new net PMID: IC5.20 (PMID)
- new net VBAT: C20.1, IC6.6 (EN), IC6.7 (IN), IC6.8 (IN)

Commit message: significant progress
Parts:
- added BT1: Battery_Cell, AA_Connectors:BH18650PC, symbol Device:Battery_Cell
- added C21: 2.2u, Capacitor_SMD:C_0805_2012Metric, symbol Device:C
- added C22, C31, C32: 1u, Capacitor_SMD:C_0805_2012Metric, symbol Device:C
- added C29: 33n, Capacitor_SMD:C_0805_2012Metric, symbol Device:C
- added C30: 22u, Capacitor_SMD:C_0805_2012Metric, symbol Device:C
- added D13: Yellow, LED_SMD:LED_0805_2012Metric, symbol Device:LED_Filled
- added L1: 1u, Inductor_SMD:L_0805_2012Metric, symbol Device:L
- added R17: 5.6k, Resistor_SMD:R_0805_2012Metric, symbol Device:R_US
- added R21: 12k, Resistor_SMD:R_0805_2012Metric, symbol Device:R_US
- added R26: 1.3k, Resistor_SMD:R_0805_2012Metric, symbol Device:R_US
- added R27: 150R, Resistor_SMD:R_0805_2012Metric, symbol Device:R_US
- added TH1: R_{0}= 10K, B = 3470K, AA_Resistors:MF52A2103J3470, symbol Device:Thermistor_NTC
- added TP33, TP34, TP35, TP36, TP37, TP38, TP39, TP40, TP41, TP42: TestPoint, AA_TestPoints:RCWCTE, symbol Connector:TestPoint
- IC5: footprint QFN50P400X400X100-25N-D -> QFN:QFN50P400X400X100-25N-D
Connections:
- net +3.3V: now also TP39.1
- net EPAD: now also IC5.15 (PGND), IC5.16 (PGND), IC5.22 (ILIM), IC5.23 (VDPM), IC5.25 (EP), IC5.4 (AGND), BT1.2 (-), C21.2, C22.2, C30.2, C31.2, C32.2, R21.2, R26.1, R26.2, TH1.2
- net PMID: now also C22.1
- net VBAT: now also IC5.13 (SYS), IC5.14 (SYS), C30.1, L1.2, TP40.1
- net VBUS: now also C21.1
- net BAT_~{CE}: now reaches IC5.1 (~{CE})
- net BAT_~{CE}: now also TP36.1
- net ISET: now reaches IC5.10 (ISET)
- net BAT+: now reaches IC5.11 (BAT), IC5.12 (BAT)
- net BAT+: now also BT1.1 (+), C32.1, TP38.1
- net SW: now reaches IC5.17 (SW), IC5.18 (SW)
- net SW: now also C29.1, L1.1
- net BAT_EN1: now reaches IC5.2 (EN1)
- net BAT_EN1: now also TP37.1
- net BOOT: now reaches IC5.21 (BOOT)
- net BOOT: now also C29.2
- net LDO: now reaches IC5.24 (LDO)
- net LDO: now also C31.1, R17.1, R27.1, TP41.1
- net BAT_EN2: now reaches IC5.3 (EN2)
- net BAT_EN2: now also TP42.1
- net PWR_SDA: now reaches IC5.5 (SDA)
- net PWR_SCL: now reaches IC5.6 (SCL)
- net STAT: now reaches IC5.7 (STAT)
- net STAT: now also D13.1 (K), TP33.1
- net BAT_INT: now reaches IC5.8 (INT)
- net BAT_INT: now also TP35.1
- net TS: now reaches IC5.9 (TS)
- net TS: now also R17.2, R21.1, TH1.1, TP34.1
- new net: D13.2 (A), R27.2
Other:
- note added: "BATTERY CHARGING"
- note added: "Battery Charge Controller"
- note added: "Battery Temperature Sensor"
- note added: "Charging Indicator"
- note added: "Decoupling"
- note added: "Default Charge Settings"
- note added: "I_{bat} maximum - 2A"
- note added: "I_{in} maximum - 2A"
- note added: "LDO for 3.3V"
- note added: "PINS TO MCU"
- note added: "POWER"
- note added: "Place thermistor next to battery"
- note added: "R_{0} = 10K B = 3470K"
- note added: "TEST POINTS"
- note added: "V_{in} minimum - 4.36V"
- moved on the sheet: C19, C20, IC5, IC6
