File: GreenNet/mcu.kicad_sch (KiCad schematic)
At the start: 31 parts, among them J2 3_Pin_Conn, J3 3_Pin_Conn, J5 3_Pin_Conn, J6 Conn_01x14_Pin, Q1 MMDT3904, SW1 SW_MEC_5E, SW3 SW_MEC_5E, U1 ESP32-S3-WROOM-1-N16R2

Commit message: layout update
Parts:
- removed D15: D5V0M1U2S9, AA_Diodes:D5V0M1U2S9Q, symbol Device:D_Zener_Filled
- removed J6: Conn_01x14_Pin, AA_Connectors:CONN_PH1-14-UA_ADM, symbol Connector:Conn_01x14_Pin
- removed R31, R32, R34: 10k, Resistor_SMD:R_0805_2012Metric, symbol Device:R_US
- added D2: D5V0M1U2S9, AA_Diodes:D5V0M1U2S9Q, symbol Device:D_Zener_Filled
- added D3: Green, LED_SMD:LED_0805_2012Metric, symbol Device:LED_Filled
- added J4: Conn_01x20_Pin, AA_Connectors:CONN_PH2-20-UA_ADM, symbol Connector:Conn_01x20_Pin
- added R11: 62R, Resistor_SMD:R_0805_2012Metric, symbol Device:R_US
- U1: value ESP32-S3-WROOM-1-N16R2 -> ESP32-S3-WROOM-1-N4R2
- renumbered C3 to C1, C1 to C2, C2 to C3, D14 to D1, J2 to J1, J3 to J2, J5 to J3, R28 to R1, R3 to R10, R1 to R2, R29 to R3, R30 to R4, R33 to R5, R2 to R9, SW3 to SW1, SW1 to SW2, TP3 to TP1, TP5 to TP2, TP31 to TP3, TP32 to TP4
Connections:
- net EPAD: now also D2.2 (A), D3.1 (K)
- net PERI_SCL: now also R5.1
- net PERI_SDA: now also R4.1
- net S3_EN_RST: now also D2.1 (K)
- net S3_IO1: now also J4.1 (Pin_1)
- net S3_IO10: now also J4.4 (Pin_4)
- net S3_IO11: now also J4.5 (Pin_5)
- net S3_IO14: now also J4.6 (Pin_6)
- net S3_IO16: now also J4.7 (Pin_7)
- net S3_IO17: now also J4.8 (Pin_8)
- net S3_IO18: now also J4.9 (Pin_9)
- net S3_IO2: now also J4.2 (Pin_2)
- net S3_IO21: now also J4.10 (Pin_10)
- net S3_IO35: now also J4.11 (Pin_11)
- net S3_IO36: now also J4.12 (Pin_12)
- net S3_IO37: now also J4.13 (Pin_13)
- net S3_IO38: now also J4.14 (Pin_14)
- net S3_IO9: now also J4.3 (Pin_3)
- net BAT_EN1 renamed S3_IO40
- net S3_IO40: now also J4.16 (Pin_16)
- net BAT_EN2 renamed S3_IO39
- net S3_IO39: now also J4.15 (Pin_15)
- net BAT_INT renamed S3_IO42
- net S3_IO42: now also J4.18 (Pin_18); no longer R4.1
- net BAT_~{CE} renamed S3_IO41
- net S3_IO41: now also J4.17 (Pin_17)
- net LCD_EN renamed LED_TEST
- net LED_TEST: now also R11.1
- net USB_GPIO renamed S3_IO48
- net S3_IO48: now also J4.20 (Pin_20)
- net USB_HPI_INT renamed S3_IO47
- net S3_IO47: now also J4.19 (Pin_19); no longer R5.1
- new net: D3.2 (A), R11.2
Other:
- note added: "Test LED"
- moved on the sheet: D1, R1, R3, R4, R5, SW1, SW2
