File: GreenNet/mcu.kicad_sch (KiCad schematic)
At the start: 30 parts, among them J1 3_Pin_Conn, J2 3_Pin_Conn, J3 3_Pin_Conn, J4 Conn_01x20_Pin, Q1 MMDT3904, SW1 SW_MEC_5E, SW2 SW_MEC_5E, U1 ESP32-S3-WROOM-1-N4R2

Commit message: update
Parts:
- removed R1: 10k, Resistor_SMD:R_0805_2012Metric, symbol Device:R_US
- added H5: MountingHole_Pad, MountingHole:MountingHole_2.5mm_Pad, symbol Mechanical:MountingHole_Pad
Connections:
- net EPAD: now also H5.1
- net LTR_INT: now also R3.1
- net PWR_SCL: no longer names the net of U1.21 (IO13)
- net PWR_SCL: no longer R3.1
- net PWR_SDA: no longer names the net of U1.20 (IO12)
- no-connect marks 0 -> 2

Commit message: update
Parts:
- TP1: value TestPoint -> PERI_SDA
- TP2: value TestPoint -> PERI_SCL
- TP3: value TestPoint -> S3_EN_RST
- TP4: value TestPoint -> S3_BOOT
Changed lines of the file:
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@@
 			)
 		)
-		(property "Value" "TestPoint"
-			(at 27.94 145.288 0)
+		(property "Value" "S3_EN_RST"
+			(at 26.416 145.288 0)
 			(effects
 				(font
@@
 			)
 		)
-		(property "Value" "TestPoint"
+		(property "Value" "PERI_SCL"
 			(at 27.94 138.938 0)
 			(effects
@@
 			)
 		)
-		(property "Value" "TestPoint"
+		(property "Value" "S3_BOOT"
 			(at 27.94 151.638 0)
 			(effects
@@
 			)
 		)
-		(property "Value" "TestPoint"
+		(property "Value" "PERI_SDA"
 			(at 27.94 132.588 0)
 			(effects
