File: GreenNet/input.kicad_sch (KiCad schematic)
At the start: 61 parts, among them J1 Conn_01x03_Pin, Q2 2N7002K, U2 AP63203WU, U3 USB_C_Receptacle_12P, U4 CP2102N-A02-GQFN28, U5 BME280, U6 USB_C_Receptacle_12P, U7 LTR-303ALS-01

Commit message: layout update
Parts:
- removed TP13: UART_VDD, AA_TestPoints:RCWCTE, symbol Connector:TestPoint
- removed TP14: VUART, AA_TestPoints:RCWCTE, symbol Connector:TestPoint
- removed TP15: VUSB, AA_TestPoints:RCWCTE, symbol Connector:TestPoint
- removed TP19, TP20: TestPoint, AA_TestPoints:RCWCTE, symbol Connector:TestPoint
- removed TP25: LCD_PWR, AA_TestPoints:RCWCTE, symbol Connector:TestPoint
- removed TP28: SOIL_PWR, AA_TestPoints:RCWCTE, symbol Connector:TestPoint
- removed TP7: LTR_INT, AA_TestPoints:RCWCTE, symbol Connector:TestPoint
- removed TP8: LCD_EN, AA_TestPoints:RCWCTE, symbol Connector:TestPoint
- D10: renamed from D7; footprint (none) -> AA_Diodes:DSS14U
- D11: renamed from D10; footprint (none) -> AA_Diodes:DSS14U
- L1: footprint (none) -> AA_Inductors:ASPI0628150MT1
- renumbered C21 to C10, C18 to C11, C13 to C12, C4 to C13, C5 to C15, C15 to C16, C6 to C17, C16 to C18, C7 to C19, C8 to C20, C11 to C4, C9 to C5, C17 to C6, C10 to C7, C12 to C8, C20 to C9, D19 to D12, D6 to D13, D1 to D4, D2 to D5, D17 to D6, D3 to D7, D18 to D8, D4 to D9, J1 to J5, R9 to R12, R4 to R13, R10 to R14, R5 to R15, R11 to R16, R8 to R17, R6 to R18, TP22 to TP10, TP23 to TP11, TP24 to TP12, TP26 to TP13, TP17 to TP5, TP18 to TP6, TP16 to TP7, TP27 to TP8, TP21 to TP9, U6 to U2, U2 to U4, U4 to U6
Connections:
- net RXT: no longer names the net of U6.18 (RXT)
- net TXT: no longer names the net of U6.19 (TXT)
- net ~{SUSPEND}: no longer names the net of U6.11 (~{SUSPEND})
- no-connect marks 17 -> 20
Other:
- note removed: "Power"
- moved on the sheet: TP10, TP11, TP12, TP13, TP5, TP6, TP7, TP8, TP9

Commit message: update
Parts:
- TP10: value TestPoint -> USB_D+
- TP11: value TestPoint -> USB_UART_D-
- TP12: value TestPoint -> USB_UART_D+
- TP5: value TestPoint -> UART_TXD
- TP6: value TestPoint -> UART_RXD
- TP9: value TestPoint -> USB_D-
Other:
- moved on the sheet: TP10, TP11, TP12, TP13, TP5, TP6, TP7, TP8, TP9
